Commit message: correct parameter

File: Project_2_GoChaseIt/my_robot/urdf/my_robot.xacro (robot description, xacro)
@@ -3,21 +3,15 @@
     <!-- CONSTANTS -->
     <xacro:property name="pi" value="3.1415926535897931" />
-    <!-- Multiplicative factor applied to the radius of the caster balls
-         for them not to stop both wheels to be touching the ground at
-         the same time                                               -->
-    <xacro:property name="reduction_factor_caster_radius" value="0.998" />
     <!-- PARAMETERS -->
+    <!-- Wheel parameters -->
+    <xacro:property name="wheel_radius" value="0.2" />
+    <xacro:property name="wheel_length" value="0.1" />
+    <xacro:property name="wheel_mass" value="5.0" />
+    <xacro:property name="z_offset_between_centers" value="${wheel_radius - base_height/30}" />
     <!-- Base parameters -->
-    <xacro:property name="base_radius" value="0.4" />
-    <!-- base height must be inside (wheel_radius, 2*wheel_radius) -->
-    <!-- note that the extremes of the interval are not included   -->
-    <xacro:property name="base_height" value="0.15" />
+    <xacro:property name="base_radius" value="0.3" />
+    <xacro:property name="base_height" value="0.6" />
     <xacro:property name="base_mass" value="15.0" />
-    <!-- Wheel parameters -->
-    <xacro:property name="wheel_radius" value="0.1" />
-    <xacro:property name="wheel_length" value="0.05" />
-    <xacro:property name="wheel_mass" value="5.0" />
-    <xacro:property name="z_offset_between_centers" value="${wheel_radius - base_height/2}" />
-    <!-- Camera parameters -->
+      <!-- Camera parameters -->
     <xacro:property name="camera_edge_length" value="0.05" />
     <xacro:property name="camera_mass" value="0.1" />
@@ -29,4 +23,5 @@
     <xacro:property name="sensors_base_mass" value="5.0" />
     <xacro:property name="sensors_base_offset_z" value="${base_height/2 + sensors_base_heigth/2}" />
+    <xacro:property name="reduction_factor_caster_radius" value="0.998" />
     <!-- INCLUDES -->
     <xacro:include filename="$(find my_robot)/urdf/materials.xacro" />
@@ -42,6 +37,4 @@
     <!-- Cylindrical base with two casters for stability along the y axis-->
     <link name="base">
-        <!-- we want the wheel to touch the ground and the top of the base
-             to coincide with the top of the wheel                       -->
         <pose>0 0 ${wheel_radius + z_offset_between_centers} 0 0 0</pose>
         <xacro:cylinder_inertial
@@ -98,6 +91,6 @@
     </link>
     <!-- Wheels on the x axis with their corresponding joints -->
+    <xacro:wheel side="right" reflect="1" />
     <xacro:wheel side="left" reflect="-1" />
-    <xacro:wheel side="right" reflect="1" />
     <!-- Rotating base for the sensors -->
     <link name="sensors_base">

Commit message: fix upper part to avid camera movement

File: Project_2_GoChaseIt/my_robot/urdf/my_robot.xacro (robot description, xacro)
@@ -111,5 +111,5 @@
         </visual>
     </link>
-    <joint name="sensors_base_hinge" type="continuous">
+    <joint name="sensors_base_hinge" type="fixed">
         <origin xyz="0 0 ${sensors_base_offset_z}" rpy="0 0 0" />
         <child link="sensors_base" />
